Commit message: URDF fix

File: urdf/makerspet_loki.urdf.xacro (robot description, xacro)
@@ -1,4 +1,4 @@
 <?xml version="1.0" ?>
-<robot name="kaia_loki" xmlns:xacro="http://ros.org/wiki/xacro">
+<robot name="makerspet_loki" xmlns:xacro="http://ros.org/wiki/xacro">
   <!-- https://classic.gazebosim.org/tutorials?tut=ros_gzplugins&cat=connect_ros -->
   <!-- https://classic.gazebosim.org/tutorials?tut=ros_urdf&cat=connect_ros -->
@@ -281,5 +281,5 @@
       <origin xyz="0 0 0" rpy="0 0 0"/>
       <geometry>
-        <mesh filename="package://kaia_loki_description/sdf/kaia_loki/mesh/head.stl" scale="${0.001*base_diameter} ${0.001*base_diameter} ${0.001*head_height*2}"/>
+        <mesh filename="package://makerspet_loki/sdf/makerspet_loki/mesh/head.stl" scale="${0.001*base_diameter} ${0.001*base_diameter} ${0.001*head_height*2}"/>
       </geometry>
       <material name="red"/>
@@ -502,5 +502,5 @@
       <plugin filename="libgazebo_ros_imu_sensor.so" name="imu_plugin">
         <ros>
-          <!-- namespace>/kaia_loki</namespace -->
+          <!-- namespace>/robot_instance_1</namespace -->
           <remapping>~/out:=imu</remapping>
         </ros>

Commit message: SDF fix

File: urdf/makerspet_loki.urdf.xacro (robot description, xacro)
@@ -281,5 +281,5 @@
       <origin xyz="0 0 0" rpy="0 0 0"/>
       <geometry>
-        <mesh filename="package://makerspet_loki/sdf/makerspet_loki/mesh/head.stl" scale="${0.001*base_diameter} ${0.001*base_diameter} ${0.001*head_height*2}"/>
+        <mesh filename="package://makerspet_loki/mesh/head.stl" scale="${0.001*base_diameter} ${0.001*base_diameter} ${0.001*head_height*2}"/>
       </geometry>
       <material name="red"/>

Commit message: URDF 200mm wheel base

File: urdf/makerspet_loki.urdf.xacro (robot description, xacro)
@@ -14,5 +14,5 @@
   <xacro:property name="floor_clearance" value="0.018"/>
   <xacro:property name="base_diameter" value="0.200"/>
-  <xacro:property name="wheel_base" value="0.131397"/>
+  <xacro:property name="wheel_base" value="0.162794"/>
   <xacro:property name="lower_cylinder_height" value="0.119"/>
   <xacro:property name="lower_to_upper_cylinders_gap" value="0.026"/>

Commit message: URDF

File: urdf/makerspet_loki.urdf.xacro (robot description, xacro)
@@ -13,12 +13,12 @@
   <xacro:property name="caster_inset" value="0.0405"/>
   <xacro:property name="floor_clearance" value="0.018"/>
-  <xacro:property name="base_diameter" value="0.200"/>
-  <xacro:property name="wheel_base" value="0.162794"/>
-  <xacro:property name="lower_cylinder_height" value="0.119"/>
-  <xacro:property name="lower_to_upper_cylinders_gap" value="0.026"/>
-  <xacro:property name="laser_puck_to_upper_cylinder_gap" value="0.005"/>
+  <xacro:property name="base_diameter" value="0.2042"/>
+  <xacro:property name="wheel_base" value="0.159063"/>
+  <xacro:property name="lower_cylinder_height" value="0.1227"/>
+  <xacro:property name="lower_to_upper_cylinders_gap" value="0.0195"/>
+  <xacro:property name="laser_puck_to_upper_cylinder_gap" value="0.0022"/>
   <xacro:property name="laser_puck_diameter" value="0.0656"/>
-  <xacro:property name="upper_cylinder_height" value="0.013"/>
-  <xacro:property name="head_height" value="0.104"/>
+  <xacro:property name="upper_cylinder_height" value="0.003"/>
+  <xacro:property name="head_height" value="0.09"/>
   <xacro:property name="tablet_width" value="0.1669"/>
   <xacro:property name="tablet_height" value="0.0781"/>
@@ -27,5 +27,5 @@
   <xacro:property name="tablet_pitch_angle" value="20"/>
   <!-- Upper cylinder's front to tablet bottom's center -->
-  <xacro:property name="tablet_inset" value="0.055"/>
+  <xacro:property name="tablet_inset" value="0.072128"/>
   <xacro:property name="color_camera_diameter" value="0.004"/>
   <!-- Tablet edge to camera center -->

Commit message: Update makerspet_loki.urdf.xacro

File: urdf/makerspet_loki.urdf.xacro (robot description, xacro)
@@ -27,5 +27,5 @@
   <xacro:property name="tablet_pitch_angle" value="20"/>
   <!-- Upper cylinder's front to tablet bottom's center -->
-  <xacro:property name="tablet_inset" value="0.072128"/>
+  <xacro:property name="tablet_inset" value="0.07"/>
   <xacro:property name="color_camera_diameter" value="0.004"/>
   <!-- Tablet edge to camera center -->

Commit message: Update makerspet_loki.urdf.xacro

File: urdf/makerspet_loki.urdf.xacro (robot description, xacro)
@@ -11,5 +11,5 @@
   <xacro:property name="caster_diameter" value="0.042"/>
   <!-- Caster center to base edge -->
-  <xacro:property name="caster_inset" value="0.0405"/>
+  <xacro:property name="caster_inset" value="0.0386"/>
   <xacro:property name="floor_clearance" value="0.018"/>
   <xacro:property name="base_diameter" value="0.2042"/>
